Commit message: Added a simple controller for Create3, commented out the URDF-parts that do not work (Possibly due to WSL)Started to work on the status communication between drones

File: src/create3_sim/irobot_create_common/irobot_create_description/urdf/catcher.urdf.xacro (robot description, xacro)
@@ -34,4 +34,7 @@
       </geometry>
     </visual>
+    <material name="green color">
+      <color rgba="11 156 49 0.8"/>
+    </material>
     <collision>
       <origin xyz="0 0 0" rpy="0 0 0"/>

File: src/create3_sim/irobot_create_common/irobot_create_description/urdf/create3.urdf.xacro (robot description, xacro)
@@ -12,5 +12,5 @@
   <xacro:include filename="$(find irobot_create_description)/urdf/wheel_with_wheeldrop.urdf.xacro" />
   <!-- Adding a link for catching the drone -->
-  <xacro:include filename="$(find irobot_create_description)/urdf/catcher.urdf.xacro" />
+  <!-- <xacro:include filename="$(find irobot_create_description)/urdf/catcher.urdf.xacro" /> -->
   <!-- Gazebo version -->
   <xacro:arg name="gazebo"                       default="classic" />
@@ -68,10 +68,10 @@
   </link>
  <!-- Adding the catcher sybassembly to the robot -->
-<xacro:catcher_subassembly
+<!-- <xacro:catcher_subassembly
     parent_link="base_link"
     catcher_xyz="0 0 0.1"
     catcher_rpy="0 0 0"
     sphere_xyz="0 0.4 0"
-    sphere_rpy="0 0 0"/>
+    sphere_rpy="0 0 0"/>  -->
   <xacro:if value="${'$(arg gazebo)' == 'ignition'}">
     <gazebo reference="base_link">

Commit message: Last version of the multithread executor concept, it seems to not work

File: src/create3_sim/irobot_create_common/irobot_create_description/urdf/catcher.urdf.xacro (robot description, xacro)
@@ -35,5 +35,5 @@
     </visual>
     <material name="green color">
-      <color rgba="11 156 49 0.8"/>
+    <color rgba="0.043 0.612 0.192 0.8"/>
     </material>
     <collision>

File: src/create3_sim/irobot_create_common/irobot_create_description/urdf/create3.urdf.xacro (robot description, xacro)
@@ -70,17 +70,18 @@
  <!--<xacro:catcher_subassembly
     parent_link="base_link"
-    catcher_xyz="0 0 0.1"
+    catcher_xyz="0 0 0.3"
     catcher_rpy="0 0 0"
-    sphere_xyz="0 0 0"
+    sphere_xyz="0 0 0.3"
     sphere_rpy="0 0 0"/> -->
    <!-- Add a green sphere for debugging -->
+   <!-- For some reason this works only at random...-->
    <link name="green_sphere_link">
   <visual>
     <origin xyz="0 0 0" rpy="0 0 0"/>
     <geometry>
-      <sphere radius="0.5"/>
+      <sphere radius="0.05"/>
     </geometry>
     <material name="green">
-      <color rgba="0 1 0 1"/>
+    <color rgba="0.043 0.612 0.192 0.8"/>
     </material>
   </visual>
@@ -92,12 +93,15 @@
   </collision>
   <inertial>
-    <mass value="1.0"/>
+    <mass value="0.0"/>
     <origin xyz="0 0 0" rpy="0 0 0"/>
     <inertia
-      ixx="0.1" ixy="0.0" ixz="0.0"
-      iyy="0.1" iyz="0.0"
-      izz="0.1"/>
+      ixx="0.0" ixy="0.0" ixz="0.0"
+      iyy="0.0" iyz="0.0"
+      izz="0.0"/>
   </inertial>
 </link>
+<gazebo reference="green_sphere_link">
+  <material>Gazebo/Green</material>
+</gazebo>
 <joint name="green_sphere_joint" type="fixed">
   <parent link="base_link"/>
