Commit message: A fight with the URDF-files. I lost

File: src/create3_sim/irobot_create_common/irobot_create_description/urdf/create3.urdf.xacro (robot description, xacro)
@@ -12,5 +12,5 @@
   <xacro:include filename="$(find irobot_create_description)/urdf/wheel_with_wheeldrop.urdf.xacro" />
   <!-- Adding a link for catching the drone -->
-  <!-- <xacro:include filename="$(find irobot_create_description)/urdf/catcher.urdf.xacro" /> -->
+   <!--<xacro:include filename="$(find irobot_create_description)/urdf/catcher.urdf.xacro" /> -->
   <!-- Gazebo version -->
   <xacro:arg name="gazebo"                       default="classic" />
@@ -68,10 +68,41 @@
   </link>
  <!-- Adding the catcher sybassembly to the robot -->
-<!-- <xacro:catcher_subassembly
+ <!--<xacro:catcher_subassembly
     parent_link="base_link"
     catcher_xyz="0 0 0.1"
     catcher_rpy="0 0 0"
-    sphere_xyz="0 0.4 0"
-    sphere_rpy="0 0 0"/>  -->
+    sphere_xyz="0 0 0"
+    sphere_rpy="0 0 0"/> -->
+   <!-- Add a green sphere for debugging -->
+   <link name="green_sphere_link">
+  <visual>
+    <origin xyz="0 0 0" rpy="0 0 0"/>
+    <geometry>
+      <sphere radius="0.5"/>
+    </geometry>
+    <material name="green">
+      <color rgba="0 1 0 1"/>
+    </material>
+  </visual>
+  <collision>
+    <origin xyz="0 0 0" rpy="0 0 0"/>
+    <geometry>
+      <sphere radius="0.5"/>
+    </geometry>
+  </collision>
+  <inertial>
+    <mass value="1.0"/>
+    <origin xyz="0 0 0" rpy="0 0 0"/>
+    <inertia
+      ixx="0.1" ixy="0.0" ixz="0.0"
+      iyy="0.1" iyz="0.0"
+      izz="0.1"/>
+  </inertial>
+</link>
+<joint name="green_sphere_joint" type="fixed">
+  <parent link="base_link"/>
+  <child link="green_sphere_link"/>
+  <origin xyz="0 0 1.5" rpy="0 0 0"/>
+</joint>
   <xacro:if value="${'$(arg gazebo)' == 'ignition'}">
     <gazebo reference="base_link">

Commit message: This might work.. But the URDF never works

File: src/create3_sim/irobot_create_common/irobot_create_description/urdf/create3.urdf.xacro (robot description, xacro)
@@ -74,6 +74,5 @@
     sphere_xyz="0 0 0.3"
     sphere_rpy="0 0 0"/> -->
-   <!-- Add a green sphere for debugging -->
-   <!-- For some reason this works only at random...-->
+   <!-- Add a green sphere -->
    <link name="green_sphere_link">
   <visual>
@@ -89,5 +88,5 @@
     <origin xyz="0 0 0" rpy="0 0 0"/>
     <geometry>
-      <sphere radius="0.5"/>
+      <sphere radius="0.05"/>
     </geometry>
   </collision>
@@ -109,4 +108,41 @@
   <origin xyz="0 0 1.5" rpy="0 0 0"/>
 </joint>
+<!-- Add a square platform for the drone to land onto -->
+  <!-- Square platform link -->
+  <link name="square_platform_link">
+    <visual>
+      <origin xyz="0 0 0" rpy="0 0 0"/>
+      <geometry>
+        <box size="1 1 0.1"/>
+      </geometry>
+      <material>
+        <color rgba="0.2 0.2 1.0 1.0"/> <!-- Blueish for visibility -->
+      </material>
+    </visual>
+    <collision>
+      <origin xyz="0 0 0" rpy="0 0 0"/>
+      <geometry>
+        <box size="1 1 0.1"/>
+      </geometry>
+    </collision>
+      <inertial>
+    <mass value="0.01"/>
+    <origin xyz="0 0 0" rpy="0 0 0"/>
+    <inertia
+      ixx="0.01" ixy="0.01" ixz="0.01"
+      iyy="0.01" iyz="0.01"
+      izz="0.01"/>
+  </inertial>
+  </link>
+  <gazebo reference="square_platform_link">
+  <cast_shadows>false</cast_shadows>
+  <material>Gazebo/Blue</material>
+  </gazebo>
+  <!-- Fixed joint to attach platform above base_link but below the sphere -->
+  <joint name="platform_joint" type="fixed">
+    <parent link="base_link"/>
+    <child link="square_platform_link"/>
+    <origin xyz="0 0 0.75" rpy="0 0 0"/>
+  </joint>
   <xacro:if value="${'$(arg gazebo)' == 'ignition'}">
     <gazebo reference="base_link">

Commit message: Small fixes, URDF is working now!

File: src/create3_sim/irobot_create_common/irobot_create_description/urdf/create3.urdf.xacro (robot description, xacro)
@@ -79,5 +79,5 @@
     <origin xyz="0 0 0" rpy="0 0 0"/>
     <geometry>
-      <sphere radius="0.05"/>
+      <sphere radius="0.03"/>
     </geometry>
     <material name="green">
@@ -88,5 +88,5 @@
     <origin xyz="0 0 0" rpy="0 0 0"/>
     <geometry>
-      <sphere radius="0.05"/>
+      <sphere radius="0.03"/>
     </geometry>
   </collision>
@@ -114,7 +114,7 @@
       <origin xyz="0 0 0" rpy="0 0 0"/>
       <geometry>
-        <box size="1 1 0.1"/>
+        <box size="0.75 0.75 0.05"/>
       </geometry>
-      <material>
+      <material name = "blue">
         <color rgba="0.2 0.2 1.0 1.0"/> <!-- Blueish for visibility -->
       </material>
@@ -123,5 +123,5 @@
       <origin xyz="0 0 0" rpy="0 0 0"/>
       <geometry>
-        <box size="1 1 0.1"/>
+        <box size="0.75 0.75 0.05"/>
       </geometry>
     </collision>
@@ -143,5 +143,5 @@
     <parent link="base_link"/>
     <child link="square_platform_link"/>
-    <origin xyz="0 0 0.75" rpy="0 0 0"/>
+    <origin xyz="0 0 0.2" rpy="0 0 0"/>
   </joint>
   <xacro:if value="${'$(arg gazebo)' == 'ignition'}">

Commit message: Cleanup and added walls to URDF-platform. Create3 should be able to continue movement now after the pause

File: src/create3_sim/irobot_create_common/irobot_create_description/urdf/create3.urdf.xacro (robot description, xacro)
@@ -67,11 +67,4 @@
     </xacro:inertial_cylinder_with_pose>
   </link>
- <!-- Adding the catcher sybassembly to the robot -->
- <!--<xacro:catcher_subassembly
-    parent_link="base_link"
-    catcher_xyz="0 0 0.3"
-    catcher_rpy="0 0 0"
-    sphere_xyz="0 0 0.3"
-    sphere_rpy="0 0 0"/> -->
    <!-- Add a green sphere -->
    <link name="green_sphere_link">
@@ -145,4 +138,105 @@
     <origin xyz="0 0 0.2" rpy="0 0 0"/>
   </joint>
+<!-- Adding some wall to the platform -->
+<link name="front_wall">
+  <visual>
+    <geometry>
+      <box size="0.73 0.01 0.1"/>
+    </geometry>
+    <origin xyz="0 0 0.02"/>
+    <material name="blue"/>
+  </visual>
+  <collision>
+    <geometry>
+      <box size="0.73 0.01 0.1"/>
+    </geometry>
+    <origin xyz="0 0 0.02"/>
+  </collision>
+  <inertial>
+    <mass value="0.0"/>
+    <origin xyz="0 0 0"/>
+    <inertia ixx="0.0" ixy="0.0" ixz="0.0" iyy="0.0" iyz="0.0" izz="0.0"/>
+  </inertial>
+</link>
+<joint name="front_wall_joint" type="fixed">
+  <parent link="square_platform_link"/>
+  <child link="front_wall"/>
+  <origin xyz="0 0.3755 0.0625" rpy="0 0 0"/>
+</joint>
+<link name="back_wall">
+  <visual>
+    <geometry>
+      <box size="0.73 0.01 0.1"/>
+    </geometry>
+    <origin xyz="0 0 0.02"/>
+    <material name="blue"/>
+  </visual>
+  <collision>
+    <geometry>
+      <box size="0.73 0.01 0.1"/>
+    </geometry>
+    <origin xyz="0 0 0.02"/>
+  </collision>
+  <inertial>
+    <mass value="0.0"/>
+    <origin xyz="0 0 0"/>
+    <inertia ixx="0.0" ixy="0.0" ixz="0.0" iyy="0.0" iyz="0.0" izz="0.0"/>
+  </inertial>
+</link>
+<joint name="back_wall_joint" type="fixed">
+  <parent link="square_platform_link"/>
+  <child link="back_wall"/>
+  <origin xyz="0 -0.3755 0.0625" rpy="0 0 0"/>
+</joint>
+<link name="left_wall">
+  <visual>
+    <geometry>
+      <box size="0.01 0.73 0.1"/>
+    </geometry>
+    <origin xyz="0 0 0.02"/>
+    <material name="blue"/>
+  </visual>
+  <collision>
+    <geometry>
+      <box size="0.01 0.73 0.1"/>
+    </geometry>
+    <origin xyz="0 0 0.02"/>
+  </collision>
+  <inertial>
+    <mass value="0.0"/>
+    <origin xyz="0 0 0"/>
+    <inertia ixx="0.0" ixy="0.0" ixz="0.0" iyy="0.0" iyz="0.0" izz="0.0"/>
+  </inertial>
+</link>
+<joint name="left_wall_joint" type="fixed">
+  <parent link="square_platform_link"/>
+  <child link="left_wall"/>
+  <origin xyz="-0.37 0 0.0625" rpy="0 0 0"/>
+</joint>
+<link name="right_wall">
+  <visual>
+    <geometry>
+      <box size="0.01 0.73 0.1"/>
+    </geometry>
+    <origin xyz="0 0 0.02"/>
+    <material name="blue"/>
+  </visual>
+  <collision>
+    <geometry>
+      <box size="0.01 0.73 0.1"/>
+    </geometry>
+    <origin xyz="0 0 0.02"/>
+  </collision>
+  <inertial>
+    <mass value="0.0"/>
+    <origin xyz="0 0 0"/>
+    <inertia ixx="0.0" ixy="0.0" ixz="0.0" iyy="0.0" iyz="0.0" izz="0.0"/>
+  </inertial>
+</link>
+<joint name="right_wall_joint" type="fixed">
+  <parent link="square_platform_link"/>
+  <child link="right_wall"/>
+  <origin xyz="0.37 0 0.0625" rpy="0 0 0"/>
+</joint>
   <xacro:if value="${'$(arg gazebo)' == 'ignition'}">
     <gazebo reference="base_link">
